File: Hardware/HA Deck 1.0/HA_Deck_v1.kicad_sch (KiCad schematic)
At the start: 28 parts, among them J1 Conn_01x03_Pin, J10 Conn_01x03_Pin, J11 Conn_01x03_Pin, J12 Conn_01x03_Pin, J13 Conn_01x03_Pin, J2 Conn_01x03_Pin, J3 Conn_01x03_Pin, J4 Conn_01x03_Pin, J5 Conn_01x03_Pin, J6 Conn_01x04_Pin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

Commit message: updated sw
Other:
- title: (none) -> Home Assistant Arcade Panel
- moved on the sheet: BZ1, DS2, J1, J10, J11, J12, J13, J2, J3, J4, J5, J6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
